Commit message: arruma os mundos e a câmera

File: src/p3dx_description/urdf/pioneer3dx_camera.xacro (robot description, xacro)
@@ -177,5 +177,5 @@
 	<joint name="camera_joint" type="fixed">
 		<axis xyz="0 1 0" />
-		<origin xyz="0 0 0.5" rpy="0 0 0"/>
+		<origin xyz="0 0 1.0" rpy="0 0.5 0"/>
 		<parent link="base_link"/>
 		<child link="camera_link"/>

Commit message: tentando adicionar a câmera rgb-d

File: src/p3dx_description/urdf/pioneer3dx_camera.xacro (robot description, xacro)
@@ -145,4 +145,5 @@
 		<child link="center_hubcap"/>
 	</joint>
+	<!-- base -->
 	<xacro:p3dx_wheel suffix="left" parent="base_link" reflect="-1"/>
 	<xacro:p3dx_wheel suffix="right" parent="base_link" reflect="1"/>
@@ -175,72 +176,79 @@
 	<!-- !!!!  <<<<<<<<< CAMERA -->
 	<!-- pelo que eu entendi, podera ir para dentro de outro .xacro ou .urdf, isso? -->
-	<joint name="camera_joint" type="fixed">
+	<!-- <joint name="camera_joint" type="fixed">
 		<axis xyz="0 1 0" />
 		<origin xyz="0 0 1.0" rpy="0 0.5 0"/>
 		<parent link="base_link"/>
 		<child link="camera_link"/>
-	  </joint>
-	  	<!-- Camera -->
-	  	<link name="camera_link">
-		<collision>
-		  	<origin xyz="0 0 0" rpy="0 0 0"/>
-		  	<geometry>
+	</joint> -->
+	<!-- Camera -->
+	<!-- <link name="camera_link">
+		<collision>
+			<origin xyz="0 0 0" rpy="0 0 0"/>
+			<geometry>
 				<box size="0 0 0"/>
-		  </geometry>
-		</collision>
-		<visual>
-		  	<origin xyz="0 0 0" rpy="0 0 0"/>
-		  	<geometry>
+			</geometry>
+		</collision>
+		<visual>
+			<origin xyz="0 0 0" rpy="0 0 0"/>
+			<geometry>
 				<box size="0 0 0"/>
-		  	</geometry>
-		  	<material name="red"/>
-		</visual>
-		<inertial>
-		  	<mass value="1e-5" />
-		  	<origin xyz="0 0 0" rpy="0 0 0"/>
-		  	<inertia ixx="1e-6" ixy="0" ixz="0" iyy="1e-6" iyz="0" izz="1e-6" />
-		</inertial>
-	  </link>
-	  <xacro:property name="camera_link" value="0.05" /> <!-- Size of square 'camera' box -->
-	  <!-- ISSO PODE IR PARA UM OUTRO GAZEBO FILE -->
-	   	<!-- camera -->
-		<gazebo reference="camera_link">
-			<sensor type="camera" name="camera1">
-			<update_rate>30.0</update_rate>
-			<camera name="head">
-				<horizontal_fov>1.3962634</horizontal_fov>
-				<image>
-				<width>800</width>
-				<height>800</height>
-				<format>R8G8B8</format>
-				</image>
-				<clip>
-				<near>0.02</near>
-				<far>300</far>
-				</clip>
-				<noise>
-				<type>gaussian</type>
-				<!-- Noise is sampled independently per pixel on each frame.
-					That pixel's noise value is added to each of its color
-					channels, which at that point lie in the range [0,1]. -->
-				<mean>0.0</mean>
-				<stddev>0.007</stddev>
-				</noise>
-			</camera>
-			<plugin name="camera_controller" filename="libgazebo_ros_camera.so">
-				<alwaysOn>true</alwaysOn>
-				<updateRate>0.0</updateRate>
-				<cameraName>rrbot/camera1</cameraName>
-				<imageTopicName>image_raw</imageTopicName>
-				<cameraInfoTopicName>camera_info</cameraInfoTopicName>
-				<frameName>camera_link</frameName>
-				<hackBaseline>0.07</hackBaseline>
-				<distortionK1>0.0</distortionK1>
-				<distortionK2>0.0</distortionK2>
-				<distortionK3>0.0</distortionK3>
-				<distortionT1>0.0</distortionT1>
-				<distortionT2>0.0</distortionT2>
-			</plugin>
-			</sensor>
-		</gazebo>
+			</geometry>
+			<material name="red"/>
+		</visual>
+		<inertial>
+			<mass value="1e-5" />
+			<origin xyz="0 0 0" rpy="0 0 0"/>
+			<inertia ixx="1e-6" ixy="0" ixz="0" iyy="1e-6" iyz="0" izz="1e-6" />
+		</inertial>
+	</link> -->
+	<!-- <xacro:property name="camera_link" value="0.05" /> --> <!-- Size of square 'camera' box -->
+	<!-- ISSO PODE IR PARA UM OUTRO GAZEBO FILE -->
+	<!-- camera -->
+	<!-- <gazebo reference="camera_link">
+		<sensor type="camera" name="camera1">
+		<update_rate>30.0</update_rate>
+		<camera name="head">
+			<horizontal_fov>1.3962634</horizontal_fov>
+			<image>
+			<width>800</width>
+			<height>800</height>
+			<format>R8G8B8</format>
+			</image>
+			<clip>
+			<near>0.02</near>
+			<far>300</far>
+			</clip>
+			<noise>
+			<type>gaussian</type>
+	-->
+			<!-- Noise is sampled independently per pixel on each frame.
+				That pixel's noise value is added to each of its color
+				channels, which at that point lie in the range [0,1]. -->
+	<!--
+			<mean>0.0</mean>
+			<stddev>0.007</stddev>
+			</noise>
+		</camera>
+		<plugin name="camera_controller" filename="libgazebo_ros_camera.so">
+			<alwaysOn>true</alwaysOn>
+			<updateRate>0.0</updateRate>
+			<cameraName>rrbot/camera1</cameraName>
+			<imageTopicName>image_raw</imageTopicName>
+			<cameraInfoTopicName>camera_info</cameraInfoTopicName>
+			<frameName>camera_link</frameName>
+			<hackBaseline>0.07</hackBaseline>
+			<distortionK1>0.0</distortionK1>
+			<distortionK2>0.0</distortionK2>
+			<distortionK3>0.0</distortionK3>
+			<distortionT1>0.0</distortionT1>
+			<distortionT2>0.0</distortionT2>
+		</plugin>
+		</sensor>
+	</gazebo> -->
+	<!-- CAMERA RGB-D INTEL D345i -->
+	<xacro:include filename="$(find realsense2_description)/urdf/_d435i.urdf.xacro"/>
+  	<xacro:sensor_d435i parent="base_link">
+    	<origin xyz="0 0 0" rpy="0 0 0"/>
+	</xacro:sensor_d435i>
 </robot>

Commit message: Adiciona no xacro a câmera RGB-D

File: src/p3dx_description/urdf/pioneer3dx_camera.xacro (robot description, xacro)
@@ -174,81 +174,9 @@
 		<child link="lms100" />
 	</joint>
-	<!-- !!!!  <<<<<<<<< CAMERA -->
-	<!-- pelo que eu entendi, podera ir para dentro de outro .xacro ou .urdf, isso? -->
-	<!-- <joint name="camera_joint" type="fixed">
-		<axis xyz="0 1 0" />
-		<origin xyz="0 0 1.0" rpy="0 0.5 0"/>
-		<parent link="base_link"/>
-		<child link="camera_link"/>
-	</joint> -->
-	<!-- Camera -->
-	<!-- <link name="camera_link">
-		<collision>
-			<origin xyz="0 0 0" rpy="0 0 0"/>
-			<geometry>
-				<box size="0 0 0"/>
-			</geometry>
-		</collision>
-		<visual>
-			<origin xyz="0 0 0" rpy="0 0 0"/>
-			<geometry>
-				<box size="0 0 0"/>
-			</geometry>
-			<material name="red"/>
-		</visual>
-		<inertial>
-			<mass value="1e-5" />
-			<origin xyz="0 0 0" rpy="0 0 0"/>
-			<inertia ixx="1e-6" ixy="0" ixz="0" iyy="1e-6" iyz="0" izz="1e-6" />
-		</inertial>
-	</link> -->
-	<!-- <xacro:property name="camera_link" value="0.05" /> --> <!-- Size of square 'camera' box -->
-	<!-- ISSO PODE IR PARA UM OUTRO GAZEBO FILE -->
-	<!-- camera -->
-	<!-- <gazebo reference="camera_link">
-		<sensor type="camera" name="camera1">
-		<update_rate>30.0</update_rate>
-		<camera name="head">
-			<horizontal_fov>1.3962634</horizontal_fov>
-			<image>
-			<width>800</width>
-			<height>800</height>
-			<format>R8G8B8</format>
-			</image>
-			<clip>
-			<near>0.02</near>
-			<far>300</far>
-			</clip>
-			<noise>
-			<type>gaussian</type>
-	-->
-			<!-- Noise is sampled independently per pixel on each frame.
-				That pixel's noise value is added to each of its color
-				channels, which at that point lie in the range [0,1]. -->
-	<!--
-			<mean>0.0</mean>
-			<stddev>0.007</stddev>
-			</noise>
-		</camera>
-		<plugin name="camera_controller" filename="libgazebo_ros_camera.so">
-			<alwaysOn>true</alwaysOn>
-			<updateRate>0.0</updateRate>
-			<cameraName>rrbot/camera1</cameraName>
-			<imageTopicName>image_raw</imageTopicName>
-			<cameraInfoTopicName>camera_info</cameraInfoTopicName>
-			<frameName>camera_link</frameName>
-			<hackBaseline>0.07</hackBaseline>
-			<distortionK1>0.0</distortionK1>
-			<distortionK2>0.0</distortionK2>
-			<distortionK3>0.0</distortionK3>
-			<distortionT1>0.0</distortionT1>
-			<distortionT2>0.0</distortionT2>
-		</plugin>
-		</sensor>
-	</gazebo> -->
 	<!-- CAMERA RGB-D INTEL D345i -->
+	<!-- <xacro:include filename="$(find realsense2_description)/urdf/_d435i.urdf.xacro"/> -->
 	<xacro:include filename="$(find realsense2_description)/urdf/_d435i.urdf.xacro"/>
-  	<xacro:sensor_d435i parent="base_link">
-    	<origin xyz="0 0 0" rpy="0 0 0"/>
+  	<xacro:sensor_d435i parent="lms100">
+		<origin xyz="0 0 0.05" rpy="0 0.2 0"/>
 	</xacro:sensor_d435i>
 </robot>

Commit message: evolução

File: src/p3dx_description/urdf/pioneer3dx_camera.xacro (robot description, xacro)
@@ -178,5 +178,5 @@
 	<xacro:include filename="$(find realsense2_description)/urdf/_d435i.urdf.xacro"/>
   	<xacro:sensor_d435i parent="lms100">
-		<origin xyz="0 0 0.05" rpy="0 0.2 0"/>
+		<origin xyz="0 0 0.8" rpy="0 0.1 0"/>
 	</xacro:sensor_d435i>
 </robot>
